File: KiCad/_saved_GRRNble.sch (KiCad schematic (older format))
At the start: 48 parts, among them J1 JST_SH_06, Q1 DMG3415U, Q2 BSS138, Q3 DMG3415U, SW1 SW_Push, SW2 SW_Push, SW3 SW_Push, U1 R5F100LJAFB, U2 BUZZER, U3 SSD1306, U4 MCP73831, U5 RN4020, U6 NJM2865F33, Y1 32.768k

Commit message: WIP (PCB)
Parts:
- BT1: footprint Connectors_Mini-Universal:MiniUniversalMate-N-LokSocket_2PinHorizontal -> misc:BatteryPad
Changed lines of the file:
@@
 F 0 "BT1" H 5300 1400 50  0000 L CNN
 F 1 "Battery_Cell" H 5300 1300 50  0000 L CNN
-F 2 "Connectors_Mini-Universal:MiniUniversalMate-N-LokSocket_2PinHorizontal" V 5200 1360 50  0001 C CNN
+F 2 "misc:BatteryPad" V 5200 1360 50  0001 C CNN
 F 3 "" V 5200 1360 50  0001 C CNN
 	1    5200 1300
